File: wearable/hw/wearable/wearable.kicad_sch (KiCad schematic)
At the start: 33 parts, among them IC1 AD627ANZ, IC2 LM4041CILPR, IC3 LM2937ET-3.3_NOPB, U2 nRF52833_QIxx, U3 LM2575-5.0BU, U4 OP1177AR, U5 OP249

Commit message: WIP final schematic
Parts:
- removed C1, C2: 2uF, symbol Device:C
- removed C3, C5: 0.1uF, symbol Device:C
- removed C4: 3.3uF, symbol Device:C
- removed C6, C7, C8: 0.015uF, symbol Device:C
- removed IC1: AD627ANZ, DIP794W56P254L959H533Q8N, symbol AD627ANZ:AD627ANZ
- removed IC2: LM4041CILPR, ECE445L:ti_LM4041CILPR, symbol ti_LM4041CILPR:LM4041CILPR
- removed R1, R2: R_US, symbol Device:R_US
- removed R10: 5.1k, symbol Device:R_US
- removed R3: 39k, symbol Device:R_US
- removed R4, R5: 1M, symbol Device:R_US
- removed R6: 1k, symbol Device:R_US
- removed R7: 200k, symbol Device:R_US
- removed R8, R9: 49k, symbol Device:R_US
- removed U1: ~, Adafruit_BNO08x:BNO080, symbol BNO085:BNO080
- removed U2: nRF52833_QIxx, Package_DFN_QFN:Nordic_AQFN-73-1EP_7x7mm_P0.5mm, symbol MCU_Nordic:nRF52833_QIxx
- removed U4: OP1177AR, Package_SO:SOIC-8_3.9x4.9mm_P1.27mm, symbol Amplifier_Operational:OP1177AR
- removed U5: OP249, Package_CSP:LFCSP-8_2x2mm_P0.5mm, symbol Amplifier_Operational:OP249
- added C10, C16, C17: ${ALTIUM_VALUE}, CAPC1005X04L, symbol Nordic Passive DB:root_2_CAP_Nordic Passive DB.DbLib
- added C10, C11, C12, C13, C9: ${ALTIUM_VALUE}, CAPC1005X04L, symbol Nordic Passive DB:root_3_CAP_Nordic Passive DB.DbLib
- added C11, C14, C15: ${ALTIUM_VALUE}, CAPC1005X04L, symbol Nordic Passive DB:root_0_CAP_Nordic Passive DB.DbLib
- added C12, C16: ${ALTIUM_VALUE}, CAPC1005X04L, symbol Nordic Passive DB:root_1_CAP_Nordic Passive DB.DbLib
- added C13, C18, C19, C9: ${ALTIUM_VALUE}, CAPC1608X06L, symbol Nordic Passive DB:root_3_CAP_Nordic Passive DB.DbLib
- added C14: ${ALTIUM_VALUE}, CAPC1608X06L, symbol Nordic Passive DB:root_1_CAP_Nordic Passive DB.DbLib
- added C20, C21: 10uF, imu:0805-NO, symbol imu-eagle-import:CAP_CERAMIC0805-NOOUTLINE
- added C22, C23, C24: 0.1uF, imu:0603-NO, symbol imu-eagle-import:CAP_CERAMIC0603_NO
- added C25, C26: 22pF, imu:0603-NO, symbol imu-eagle-import:CAP_CERAMIC0603_NO
- added CONN3, CONN4: STEMMA_I2C_QT, imu:JST_SH4, symbol imu-eagle-import:STEMMA_I2C_QT
- added D2: GREEN, imu:CHIPLED_0603_NOOUTLINE, symbol imu-eagle-import:LED0603_NOOUTLINE
- added FID3, FID4: FIDUCIAL_1MM, imu:FIDUCIAL_1MM, symbol imu-eagle-import:FIDUCIAL_1MM
- added JP1, JP2: HEADER-1X670MIL, imu:1X06_ROUND_70, symbol imu-eagle-import:HEADER-1X670MIL
- added L2 (x2): ${ALTIUM_VALUE}, INDC1005X04L, symbol Nordic Passive DB:root_0_IND_Nordic Passive DB.DbLib
- added Q2: BSS138, imu:SOT363, symbol imu-eagle-import:MOSFET-N_DUAL
- added R11: ${ALTIUM_VALUE}, RESC1005X04L, symbol AltiumLib:root_0_RES_AltiumLib.DbLib
- added R12, R13, R14, R15: 10K, symbol Device:R_US
- added R16, R17, R18: 10K, imu:RESPACK_4X0603, symbol imu-eagle-import:RESISTOR_4PACK
- added SJ1: PS1, imu:SOLDERJUMPER_ARROW_NOPASTE, symbol imu-eagle-import:SOLDERJUMPER
- added SJ2: PS0, imu:SOLDERJUMPER_ARROW_NOPASTE, symbol imu-eagle-import:SOLDERJUMPER
- added U$1, U$17, U$19, U$21: MOUNTINGHOLE2.5, imu:MOUNTINGHOLE_2.5_PLATED, symbol imu-eagle-import:MOUNTINGHOLE2.5
- added U1: AP2112K-3.3, imu:SOT23-5, symbol imu-eagle-import:VREG_SOT23-5
- added U1: BNO080, imu:BNO080, symbol imu-eagle-import:BNO080
- added U2: ${ALTIUM_VALUE}, AQFN50P700X700X85_HS-74N, symbol Nordic Active DB:root_0_nRF52833_QIAA_Nordic Active DB.DbLib
- added U5: ADS1299IPAG, PAG64_TEX, symbol ADS1299:ADS1299IPAG
- added U6: 74AHC4050, imu:TSSOP16, symbol imu-eagle-import:74HC4050DTSSOP
- added X1: ${ALTIUM_VALUE}, BT-XTAL_2016, symbol Nordic Discrete DB:root_1_XTAL_4-pin_grounded_Nordic Discrete DB.DbLib
- added X2: ${ALTIUM_VALUE}, XTAL_3215, symbol Nordic Discrete DB:root_3_XTAL_2-pin_Nordic Discrete DB.DbLib
- added X3: 32.768, imu:XTAL3215, symbol imu-eagle-import:XTAL-3.2X1.5
Connections:
- net 3.3V: now also C21.1, C22.1, C23.1, JP1.2, Q2.2 (G), Q2.5 (G), R16.5 (2), R18.3 (1), R18.5 (2), U1.28 (VDDIO), U1.3 (VDD), U1.5 (OUT), U6.1 (VCC)
- net GND: now also C10.1, C10.2, C11.2, C11.2, C12.1, C12.2, C13.2, C13.2, C14.1, C14.2, C15.2, C16.1, C16.2, C17.2, C18.2, C19.2, C20.2, C21.2, C22.2, C23.2, C24.1, C25.2, C26.2, C9.2, C9.2, CONN3.1 (GND), CONN3.MT1 (MT), CONN3.MT2 (MT), CONN4.1 (GND), CONN4.MT1 (MT), CONN4.MT2 (MT), D2.C, JP1.3, R12.2, R13.2, R14.2, R15.2, R16.7 (2), R16.8 (2), R18.1, R18.2 (1), R18.8 (2), U1.10 (CLKSEL0), U1.2 (GND), U1.2 (GND), U1.25 (GNDIO), U2.74 (VSS), U2.B7 (VSS), U2.F23 (VSS_PA), U6.8 (GND)
- new net: C19.1, U2.AC5 (DECUSB)
- new net: C12.2, L2.1, U2.H23 (ANT)
- new net: C9.1, U2.N24 (DEC5)
- new net: C16.2, L2.1, L2.2
- new net: D2.A, R16.4 (1)
- new net: R12.1, U5.46 (GPIO4)
- new net: U5.31 (RESV1), U5.33 (DGND)
- new net: R15.1, U5.42 (GPIO1)
- new net: R14.1, U5.44 (GPIO2)
- new net: R13.1, U5.45 (GPIO3)
- new net BOOT: JP2.1, R16.3 (1), U6.7 (3A)
- new net BOOT_3V: U1.4 (BOOTN), U6.6 (3Y)
- new net CAP: C24.2, U1.9 (CAP)
- new net CS: JP2.6, R17.1, U6.9 (4A)
- new net CS_3V: U1.18 (H_CSN), U6.10 (4Y)
- new net D+: U2.AD6 (D+)
- new net D-: U2.AD4 (D-)
- new net DEC1: C10.1, U2.C1 (DEC1)
- new net DEC3: C11.1, U2.D23 (DEC3)
- new net DEC4_6: C10.2, C14.2, U2.B5 (DEC4), U2.E24 (DEC6)
- new net INT: JP1.6, U1.14 (H_INTN)
- new net MOSI: JP2.5, R18.7 (2), U6.11 (5A)
- new net MOSI_3V: U1.17 (H_SA0/MOSI), U6.12 (5Y)
- new net P0.00/XL1: C16.1, U2.D2 (P0.00/XL1), X2.1 (inp)
- new net P0.01/XL2: C17.1, U2.F2 (P0.01/XL2), X2.2 (out)
- new net P0.02/AIN0: U2.A12 (P0.02/AIN0)
- new net P0.03/AIN1: U2.B13 (P0.03/AIN1)
- new net P0.04/AIN2: U2.J1 (P0.04/AIN2)
- new net P0.05/AIN3: U2.K2 (P0.05/AIN3)
- new net P0.06: U2.L1 (P0.06)
- new net P0.07: U2.M2 (P0.07)
- new net P0.08: U2.N1 (P0.08)
- new net P0.09/NFC1: U2.L24 (P0.09/NFC1)
- new net P0.10/NFC2: U2.J24 (P0.10/NFC2)
- new net P0.11: U2.T2 (P0.11)
- new net P0.12: U2.U1 (P0.12)
- new net P0.13: U2.AD8 (P0.13)
- new net P0.14: U2.AC9 (P0.14)
- new net P0.15: U2.AD10 (P0.15)
- new net P0.16: U2.AC11 (P0.16)
- new net P0.17: U2.AD12 (P0.17)
- new net P0.18/RESET: U2.AC13 (P0.18/RESET)
- new net P0.19: U2.A14 (P0.19)
- new net P0.20: U2.AD16 (P0.20)
- new net P0.21: U2.AC17 (P0.21)
- new net P0.22: U2.AD18 (P0.22)
- new net P0.23: U2.B17 (P0.23)
- new net P0.24: U2.AD20 (P0.24)
- new net P0.25: U2.A20 (P0.25)
- new net P0.26: U2.G1 (P0.26)
- new net P0.27: U2.H2 (P0.27)
- new net P0.28/AIN4: U2.B11 (P0.28/AIN4)
- new net P0.29/AIN5: U2.A10 (P0.29/AIN5)
- new net P0.30/AIN6: U2.B9 (P0.30/AIN6)
- new net P0.31/AIN7: U2.A8 (P0.31/AIN7)
- new net P1.00: U2.AD22 (P1.00)
- new net P1.01: U2.Y23 (P1.01)
- new net P1.02: U2.W24 (P1.02)
- new net P1.03: U2.B15 (P1.03)
- new net P1.04: U2.U24 (P1.04)
- new net P1.05: U2.A16 (P1.05)
- new net P1.06: U2.R24 (P1.06)
- new net P1.07: U2.P23 (P1.07)
- new net P1.08: U2.P2 (P1.08)
- new net P1.09: U2.R1 (P1.09)
- new net PS0: JP2.2, R16.2 (1), SJ2.2, U6.3 (1A)
- new net PS0_3V: U1.6 (PS0/WAKE), U6.2 (1Y)
- new net PS1: JP2.3, R16.1, SJ1.2, U6.5 (2A)
- new net PS1_3V: U1.5 (PS1), U6.4 (2Y)
- new net RF: L2.2
- new net RST: JP2.4, R17.2 (1), U6.14 (6A)
- new net RST_3V: U1.11 (NRST), U6.15 (6Y)
- new net SCL/SCK/RX: CONN3.4 (SCL), CONN4.4 (SCL), JP1.4, Q2.6 (D), R17.4 (1)
- new net SCL_3V: Q2.1 (S), R18.4 (1), U1.19 (H_SCL/SCLK/RX)
- new net SDA/MISO/TX: CONN3.3 (SDA), CONN4.3 (SDA), JP1.5, Q2.3 (D), R17.3 (1)
- new net SDA_3V: Q2.4 (S), R18.6 (2), U1.20 (H_SDA/MISO/TX)
- new net SWDCLK: U2.AA24 (SWDCLK)
- new net SWDIO: U2.AC24 (SWDIO)
- new net VBUS: R11.1
- new net VBUS_nRF: C18.1, R11.2, U2.AD2 (VBUS), U2.Y2 (VDDH)
- new net VCC: C20.1, CONN3.2 (V+), CONN4.2 (V+), JP1.1, R16.6 (2), R17.5 (2), R17.6 (2), R17.7 (2), R17.8 (2), SJ1.1, SJ2.1, U1.1 (IN), U1.3 (EN)
- new net VDD_nRF: C11.1, C12.1, C13.1, C13.1, C9.1, U2.A22 (VDD), U2.AD14 (VDD), U2.AD23 (VDD), U2.B1 (VDD), U2.W1 (VDD)
- new net XC1: C15.1, U2.B24 (XC1), X1.1 (inp)
- new net XC2: C14.1, U2.A23 (XC2), X1.3 (out)
- new net XIN: C25.1, U1.27 (XIN32), X3.P$1
- new net XOUT: C26.1, U1.26 (CLKSEL1/XOUT32), X3.P$2
- no-connect marks 80 -> 12
Other:
- note added: "Close PS1 for UART Close PS1 and PS0 for SPI"
- note added: "D"
- note added: "Default Bus = I2C"
- note added: "EEG Circuit"
- note added: "G"
- note added: "I2C Pullups & Shift (IMU Breakout)"
- note added: "IMU Breakout"
- note added: "ON LED"
- note added: "Optional"
- note added: "Power Supply (Main)"
- note added: "Power supply (IMU breakout)"
- note added: "S"
- note added: "SA0 is default low, so I2C ADDR = 1001010 (0x4A)"
- note added: "STEMMA/I2C Headers (IMU Breakout)"
- note added: "nRF52833-QIAA"
- moved on the sheet: BT1, D1, IC3, L1, U3, power_C1, power_C2, power_C3, power_C4

Commit message: Done with M3 schematic
Parts:
- added C1, C27, C29, C3, C5, C7: 1uF, symbol Device:C
- added C2: 100uF, symbol Device:C
- added C28: .1uF, symbol Device:C
- added C30: 1.5nF, symbol Device:C
- added C4, C6: 0.1uF, symbol Device:C
- added C8: 10uF, symbol Device:C
- added E1, E2, E3, E4, E6: ~, symbol wearable:EEG_Electrode
- added IC1: LM4041CILPR, ECE445L:ti_LM4041CILPR, symbol ti_LM4041CILPR:LM4041CILPR
- added R1: 5.1K, symbol Device:R_US
- added R2: 1M, symbol Device:R_US
Connections:
- net MOSI_3V is gone; now on net MOSI: U1.17 (H_SA0/MOSI), U6.12 (5Y)
- net P0.19 is gone; now on net CS_ADS1299: U2.A14 (P0.19)
- net P0.23 is gone; now on net CS_BNO085: U2.B17 (P0.23)
- net P0.27 is gone; now on net SCK: U2.H2 (P0.27)
- net P0.29/AIN5 is gone; now on net MOSI: U2.A10 (P0.29/AIN5)
- net P0.31/AIN7 is gone; now on net MISO: U2.A8 (P0.31/AIN7)
- net P1.03 is gone; now on net DRDY: U2.B15 (P1.03)
- net SCL_3V is gone; now on net SCK: Q2.1 (S), R18.4 (1), U1.19 (H_SCL/SCLK/RX)
- net SDA_3V is gone; now on net MISO: Q2.4 (S), R18.6 (2), U1.20 (H_SDA/MISO/TX)
- net 3.3V: now also U5.48 (DVDD), U5.50 (DVDD), U5.52 (CLKSEL), R1.1
- net AVDD: now also U5.1 (IN8N), U5.10 (IN4P), U5.11 (IN3N), U5.12 (IN3P), U5.17 (SRB1), U5.18 (SRB2), U5.19 (AVDD), U5.2 (IN8P), U5.21 (AVDD), U5.22 (AVDD), U5.3 (IN7N), U5.4 (IN7P), U5.5 (IN6N), U5.56 (AVDD), U5.59 (AVDD), U5.6 (IN6P), U5.7 (IN5N), U5.8 (IN5P), U5.9 (IN4N), C4.1, C5.1, C6.1, C7.1
- net AVSS: now also U5.20 (AVSS), U5.23 (AVSS), U5.57 (AVSS), U5.58 (AVSS), C1.1, C2.2, C27.2, C28.2, C3.2, C4.2, C5.2, C6.2, C7.2
- net GND: now also U5.31 (RESV1), U5.33 (DGND), U5.49 (DGND), U5.51 (DGND), IC1.1, IC1.3
- net MOSI: now also U5.34 (DIN)
- net at U5.13 (IN2N): now also E1.
- net at U5.14 (IN2P): now also E2.
- net at U5.15 (IN1N): now also E3.
- net at U5.16 (IN1P): now also E4.
- net at U5.24 (VREFP): now also C8.1, IC1.2, R1.2
- net at U5.25 (VREFN): now also C8.2
- net at U5.26 (VCAP4): now also C3.1
- net at U5.28 (VCAP1): now also C2.1
- net at U5.30 (VCAP2): now also C1.2
- net PWDWN_ADS1299: now reaches U5.35 (*PWDN)
- net RST_ADS1299: now reaches U5.36 (*RESET)
- net START_ADS1299: now reaches U5.38 (START)
- net CS_ADS1299: now reaches U5.39 (*CS)
- net SCK: now reaches U5.40 (SCLK)
- net MISO: now reaches U5.43 (DOUT)
- net DRDY: now reaches U5.47 (*DRDY)
- net at U5.53 (AVSS1): now also C29.1
- net at U5.54 (AVDD1): now also C29.2
- net at U5.55 (VCAP3): now also C27.1, C28.1
- net at U5.62 (BIASIN): now also U5.63 (BIASOUT), C30.1, R2.1
- net BOOT_3V renamed BOOT_BNO085
- net CS_3V renamed CS_BNO085
- net INT renamed INT_BNO085
- net PS0_3V renamed WAKE_BNO085
- net RST_3V renamed RST_BNO085
- new net: C30.2, E6., R2.2
Other:
- note added: "(1) Set the two-state mode setting pins high to DVDD or low to DGND through ≥10-kΩ resistors."
- note added: "EEG Inputs"
- note added: "Sleep Wearable"
- note removed: "Sleep Wearable Prototype"
- moved on the sheet: C23, R12, R13, R14, R15

Commit message: Moved around some stuff
Connections:
- net P0.13 is gone; now on net START_ADS1299: U2.AD8 (P0.13)
- net P0.14 is gone; now on net RST_ADS1299: U2.AC9 (P0.14)
- net P0.15 is gone; now on net PWDWN_ADS1299: U2.AD10 (P0.15)
- net P0.16 is gone; now on net BOOT_BNO085: U2.AC11 (P0.16)
- net P0.17 is gone; now on net WAKE_BNO085: U2.AD12 (P0.17)
- net AVSS: now also U5.32 (AVSS)
- no-connect marks 12 -> 15
Other:
- note removed: "(1) Set the two-state mode setting pins high to DVDD or low to DGND through ≥10-kΩ resistors."
- moved on the sheet: E1, E2, E3, E4
Changed lines of the file:
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@@
 		)
 	)
-	(text "(1) Set the two-state mode setting pins high to DVDD \nor low to DGND through ≥10-kΩ resistors."
-		(exclude_from_sim no)
-		(at 360.172 197.612 0)
-		(effects
-			(font
-				(size 1.27 1.27)
-			)
-			(justify left)
-		)
-	)
 	(text "EEG Circuit"
 		(exclude_from_sim no)
@@
 	)
 	(no_connect
+		(at 113.665 161.925)
+	)
+	(no_connect
 		(at 342.265 231.775)
 	)
@@
 	)
 	(no_connect
+		(at 103.505 161.925)
+	)
+	(no_connect
 		(at 113.665 83.185)
 	)
 	(no_connect
+		(at 118.745 161.925)
+	)
+	(no_connect
 		(at 60.325 141.605)
 	)
@@
 	(wire
 		(pts
-			(xy 240.665 193.675) (xy 271.145 193.675)
+			(xy 238.125 193.675) (xy 271.145 193.675)
 		)
 		(stroke
@@
 	(wire
 		(pts
-			(xy 234.95 198.755) (xy 271.145 198.755)
+			(xy 232.41 198.755) (xy 271.145 198.755)
 		)
 		(stroke
@@
 	(wire
 		(pts
-			(xy 237.49 196.215) (xy 271.145 196.215)
+			(xy 234.95 196.215) (xy 271.145 196.215)
 		)
 		(stroke
@@
 	(wire
 		(pts
-			(xy 232.41 201.295) (xy 271.145 201.295)
+			(xy 229.87 201.295) (xy 271.145 201.295)
 		)
 		(stroke
@@
 		)
 	)
+	(global_label "RST_ADS1299"
+		(shape output)
+		(at 88.265 175.895 270)
+		(fields_autoplaced yes)
+		(effects
+			(font
+				(size 1.27 1.27)
+			)
+			(justify right)
+		)
+		(property "Intersheetrefs" "${INTERSHEET_REFS}"
+			(at 88.265 191.701 90)
+			(effects
+				(font
+					(size 1.27 1.27)
+				)
+				(justify right)
+				(hide yes)
+			)
+		)
+	)
 	(global_label "CS_BNO085"
 		(shape output)
@@
 		)
 	)
+	(global_label "START_ADS1299"
+		(shape output)
+		(at 85.725 175.895 270)
+		(fields_autoplaced yes)
+		(effects
+			(font
+				(size 1.27 1.27)
+			)
+			(justify right)
+		)
+		(property "Intersheetrefs" "${INTERSHEET_REFS}"
+			(at 85.725 193.7572 90)
+			(effects
+				(font
+					(size 1.27 1.27)
+				)
+				(justify right)
+				(hide yes)
+			)
+		)
+	)
 	(global_label "AVDD"
 		(shape input)
@@
 		)
 	)
+	(global_label "BOOT_BNO085"
+		(shape output)
+		(at 93.345 175.895 270)
+		(fields_autoplaced yes)
+		(effects
+			(font
+				(size 1.27 1.27)
+			)
+			(justify right)
+		)
+		(property "Intersheetrefs" "${INTERSHEET_REFS}"
+			(at 93.345 192.3059 90)
+			(effects
+				(font
+					(size 1.27 1.27)
+				)
+				(justify right)
+				(hide yes)
+			)
+		)
+	)
 	(global_label "AVSS"
 		(shape input)
@@
 		)
 	)
+	(global_label "WAKE_BNO085"
+		(shape output)
+		(at 95.885 175.895 270)
+		(fields_autoplaced yes)
+		(effects
+			(font
+				(size 1.27 1.27)
+			)
+			(justify right)
+		)
+		(property "Intersheetrefs" "${INTERSHEET_REFS}"
+			(at 95.885 192.3663 90)
+			(effects
+				(font
+					(size 1.27 1.27)
+				)
+				(justify right)
+				(hide yes)
+			)
+		)
+	)
 	(global_label "START_ADS1299"
 		(shape input)
@@
 		)
 	)
+	(global_label "PWDWN_ADS1299"
+		(shape output)
+		(at 90.805 175.895 270)
+		(fields_autoplaced yes)
+		(effects
+			(font
+				(size 1.27 1.27)
+			)
+			(justify right)
+		)
+		(property "Intersheetrefs" "${INTERSHEET_REFS}"
+			(at 90.805 195.0272 90)
+			(effects
+				(font
+					(size 1.27 1.27)
+				)
+				(justify right)
+				(hide yes)
+			)
+		)
+	)
 	(global_label "SCK"
 		(shape input)
@@
 		)
 	)
+	(global_label "AVSS"
+		(shape input)
+		(at 271.145 241.935 180)
+		(fields_autoplaced yes)
+		(effects
+			(font
+				(size 1.27 1.27)
+			)
+			(justify right)
+		)
+		(property "Intersheetrefs" "${INTERSHEET_REFS}"
+			(at 263.5636 241.935 0)
+			(effects
+				(font
+					(size 1.27 1.27)
+				)
+				(justify right)
+				(hide yes)
+			)
+		)
+	)
 	(global_label "MISO"
 		(shape output)
@@
 	(symbol
 		(lib_id "wearable:EEG_Electrode")
-		(at 231.14 198.755 0)
+		(at 228.6 198.755 0)
 		(unit 1)
 		(exclude_from_sim no)
@@
 		(fields_autoplaced yes)
 		(property "Reference" "E3"
-			(at 231.14 194.945 0)
+			(at 228.6 194.945 0)
 			(effects
 				(font
@@
 		)
 		(property "Value" "~"
-			(at 231.14 198.755 0)
+			(at 228.6 198.755 0)
 			(effects
 				(font
@@
 		)
 		(property "Footprint" ""
-			(at 231.14 198.755 0)
+			(at 228.6 198.755 0)
 			(effects
 				(font
@@
 		)
 		(property "Datasheet" ""
-			(at 231.14 198.755 0)
+			(at 228.6 198.755 0)
 			(effects
 				(font
@@
 		)
 		(property "Description" ""
-			(at 231.14 198.755 0)
+			(at 228.6 198.755 0)
 			(effects
 				(font
@@
 	(symbol
 		(lib_id "wearable:EEG_Electrode")
-		(at 233.68 196.215 0)
+		(at 231.14 196.215 0)
 		(unit 1)
 		(exclude_from_sim no)
@@
 		(fields_autoplaced yes)
 		(property "Reference" "E2"
-			(at 233.68 192.405 0)
+			(at 231.14 192.405 0)
 			(effects
 				(font
@@
 		)
 		(property "Value" "~"
-			(at 233.68 196.215 0)
+			(at 231.14 196.215 0)
 			(effects
 				(font
@@
 		)
 		(property "Footprint" ""
-			(at 233.68 196.215 0)
+			(at 231.14 196.215 0)
 			(effects
 				(font
@@
 		)
 		(property "Datasheet" ""
-			(at 233.68 196.215 0)
+			(at 231.14 196.215 0)
 			(effects
 				(font
@@
 		)
 		(property "Description" ""
-			(at 233.68 196.215 0)
+			(at 231.14 196.215 0)
 			(effects
 				(font
@@
 	(symbol
 		(lib_id "wearable:EEG_Electrode")
-		(at 236.855 193.675 0)
+		(at 234.315 193.675 0)
 		(unit 1)
 		(exclude_from_sim no)
@@
 		(fields_autoplaced yes)
 		(property "Reference" "E1"
-			(at 236.855 189.865 0)
+			(at 234.315 189.865 0)
 			(effects
 				(font
@@
 		)
 		(property "Value" "~"
-			(at 236.855 193.675 0)
+			(at 234.315 193.675 0)
 			(effects
 				(font
@@
 		)
 		(property "Footprint" ""
-			(at 236.855 193.675 0)
+			(at 234.315 193.675 0)
 			(effects
 				(font
@@
 		)
 		(property "Datasheet" ""
-			(at 236.855 193.675 0)
+			(at 234.315 193.675 0)
 			(effects
 				(font
@@
 		)
 		(property "Description" ""
-			(at 236.855 193.675 0)
+			(at 234.315 193.675 0)
 			(effects
 				(font
@@
 	(symbol
 		(lib_id "wearable:EEG_Electrode")
-		(at 228.6 201.295 0)
+		(at 226.06 201.295 0)
 		(unit 1)
 		(exclude_from_sim no)
@@
 		(fields_autoplaced yes)
 		(property "Reference" "E4"
-			(at 228.6 197.485 0)
+			(at 226.06 197.485 0)
 			(effects
 				(font
@@
 		)
 		(property "Value" "~"
-			(at 228.6 201.295 0)
+			(at 226.06 201.295 0)
 			(effects
 				(font
@@
 		)
 		(property "Footprint" ""
-			(at 228.6 201.295 0)
+			(at 226.06 201.295 0)
 			(effects
 				(font
@@
 		)
 		(property "Datasheet" ""
-			(at 228.6 201.295 0)
+			(at 226.06 201.295 0)
 			(effects
 				(font
@@
 		)
 		(property "Description" ""
-			(at 228.6 201.295 0)
+			(at 226.06 201.295 0)
 			(effects
 				(font

Commit message: HW v1 complete
Parts:
- removed C10, C16, C17: ${ALTIUM_VALUE}, CAPC1005X04L, symbol Nordic Passive DB:root_2_CAP_Nordic Passive DB.DbLib
- removed C10, C11, C12, C13, C9: ${ALTIUM_VALUE}, CAPC1005X04L, symbol Nordic Passive DB:root_3_CAP_Nordic Passive DB.DbLib
- removed C11, C14, C15: ${ALTIUM_VALUE}, CAPC1005X04L, symbol Nordic Passive DB:root_0_CAP_Nordic Passive DB.DbLib
- removed C12, C16: ${ALTIUM_VALUE}, CAPC1005X04L, symbol Nordic Passive DB:root_1_CAP_Nordic Passive DB.DbLib
- removed C13, C18, C19, C9: ${ALTIUM_VALUE}, CAPC1608X06L, symbol Nordic Passive DB:root_3_CAP_Nordic Passive DB.DbLib
- removed C14: ${ALTIUM_VALUE}, CAPC1608X06L, symbol Nordic Passive DB:root_1_CAP_Nordic Passive DB.DbLib
- removed C20, C21: 10uF, imu:0805-NO, symbol imu-eagle-import:CAP_CERAMIC0805-NOOUTLINE
- removed C22, C23, C24: 0.1uF, imu:0603-NO, symbol imu-eagle-import:CAP_CERAMIC0603_NO
- removed C25, C26: 22pF, imu:0603-NO, symbol imu-eagle-import:CAP_CERAMIC0603_NO
- removed CONN3, CONN4: STEMMA_I2C_QT, imu:JST_SH4, symbol imu-eagle-import:STEMMA_I2C_QT
- removed D1: MBR360, DIOAD2860W130L840D505, symbol MBR360:MBR360
- removed D2: GREEN, imu:CHIPLED_0603_NOOUTLINE, symbol imu-eagle-import:LED0603_NOOUTLINE
- removed IC3: LM2937ET-3.3_NOPB, ECE445L:TO254P470X1028X1955-3P, symbol ECE445L:LM2937ET-3.3_NOPB
- removed L2 (x2): ${ALTIUM_VALUE}, INDC1005X04L, symbol Nordic Passive DB:root_0_IND_Nordic Passive DB.DbLib
- removed Q2: BSS138, imu:SOT363, symbol imu-eagle-import:MOSFET-N_DUAL
- removed R11: ${ALTIUM_VALUE}, RESC1005X04L, symbol AltiumLib:root_0_RES_AltiumLib.DbLib
- removed R16, R17, R18: 10K, imu:RESPACK_4X0603, symbol imu-eagle-import:RESISTOR_4PACK
- removed SJ1: PS1, imu:SOLDERJUMPER_ARROW_NOPASTE, symbol imu-eagle-import:SOLDERJUMPER
- removed SJ2: PS0, imu:SOLDERJUMPER_ARROW_NOPASTE, symbol imu-eagle-import:SOLDERJUMPER
- removed U1: AP2112K-3.3, imu:SOT23-5, symbol imu-eagle-import:VREG_SOT23-5
- removed U1: BNO080, imu:BNO080, symbol imu-eagle-import:BNO080
- removed U3: LM2575-5.0BU, Package_TO_SOT_SMD:TO-263-5_TabPin3, symbol Regulator_Switching:LM2575-5.0BU
- removed U6: 74AHC4050, imu:TSSOP16, symbol imu-eagle-import:74HC4050DTSSOP
- removed X2: ${ALTIUM_VALUE}, XTAL_3215, symbol Nordic Discrete DB:root_3_XTAL_2-pin_Nordic Discrete DB.DbLib
- removed X3: 32.768, imu:XTAL3215, symbol imu-eagle-import:XTAL-3.2X1.5
- removed power_C1: 100uF, symbol Device:C_Polarized
- removed power_C2: 220uF, symbol Device:C_Polarized
- removed power_C3, power_C4: 4.7uF, ECE445L:CP_Radial_Tantal200mil, symbol ECE445L:C_Polarized
- added C10: NC, ECE445L:C_Axial_200mil, symbol ECE445L:C
- added C11: 820pF, ECE445L:C_Axial_200mil, symbol ECE445L:C
- added C12: 100pF, ECE445L:C_Axial_200mil, symbol ECE445L:C
- added C13: 1.2pF, ECE445L:C_Axial_200mil, symbol ECE445L:C
- added C14, C16, C43, C9: 12pF, ECE445L:C_Axial_200mil, symbol ECE445L:C
- added C15, C18, C34, C42: 100nF, ECE445L:C_Axial_200mil, symbol ECE445L:C
- added C17, C19, C20, C21, C41: 1uF, ECE445L:C_Axial_200mil, symbol ECE445L:C
- added C31: C, ECE445L:C_Axial_200mil, symbol ECE445L:C
- added C32, C35, C36, C40: 4.7uF, ECE445L:C_Axial_200mil, symbol ECE445L:C
- added C33: 47uF, ECE445L:C_Axial_200mil, symbol ECE445L:C
- added C37, C38: 22uF, ECE445L:C_Axial_200mil, symbol ECE445L:C
- added C39: 10nF, ECE445L:C_Axial_200mil, symbol ECE445L:C
- added C44: 1pF, ECE445L:C_Axial_200mil, symbol ECE445L:C
- added J8: USBC, Connector_PinHeader_2.54mm:PinHeader_1x08_P2.54mm_Vertical, symbol ECE445L:Conn_01x08_Pin
- added L3: 2.2nH, symbol Device:L
- added L4: 4.7nH, symbol Device:L
- added R3, R4: 100K, symbol Device:R_US
- added SW1: SW_Toggle, symbol Switch:SW_Push
- added U4: MAX77659AENV+, 21-100509_N302D2+1_MXM, symbol MAX77659:MAX77659AENV+
- added X2: 32.768kHz, symbol nrf52833dk:root_3_XTAL_2-pin
- L1: value 330uF -> 1.5uH
Connections:
- net BOOT is gone; now on net BOOT_BNO085: JP2.1
- net CS is gone; now on net CS_BNO085: JP2.6
- net PS0 is gone; now on net WAKE_BNO085: JP2.2
- net RST is gone; now on net RST_BNO085: JP2.4
- net SCL/SCK/RX is gone; now on net SCK: JP1.4
- net SDA/MISO/TX is gone; now on net MISO: JP1.5
- net VBUS_nRF is gone; now on net 3.3V: U2.AD2 (VBUS), U2.Y2 (VDDH)
- net VDD_nRF is gone; now on net 3.3V: U2.A22 (VDD), U2.AD14 (VDD), U2.AD23 (VDD), U2.B1 (VDD), U2.W1 (VDD)
- net 3.3V: now also C15.1, C34.1, C35.1, C36.1, C37.1, C38.1, C41.1, C42.1, R3.2, R4.2, U4.B1 (SYS), U4.C2 (IN_SBB), U4.C3 (SBB3_CHG), U4.C6 (VIO); no longer JP1.2
- net 5V: now also C33.2, J8.2 (Pin_2), U4.C1 (CHGIN); no longer L1.2
- net DEC1: now also C18.1
- net DEC3: now also C12.2
- net DEC4_6: now also C10.2, C19.1
- net GND: now also C10.1, C11.1, C12.1, C13.2, C14.1, C15.2, C16.1, C17.2, C18.2, C19.2, C20.2, C21.2, C31.2, C32.2, C33.1, C34.2, C35.2, C36.2, C37.2, C38.2, C40.2, C41.2, C42.2, C43.1, C44.1, C9.1, J8.1 (Pin_1), SW1.1, U4.A3 (THM), U4.B4 (GND), U4.E1 (PGND), U4.E5 (IN_LDO), U4.E6 (LDO)
- net P0.00/XL1: now also C9.2, X2.1 (inp)
- net P0.01/XL2: now also C16.2, X2.2 (out)
- net RF: now also L3.2
- net XC1: now also C14.2
- net XC2: now also C43.2
- net at U2.AC5 (DECUSB): now also C40.1
- net at U2.H23 (ANT): now also C44.2, L4.1
- net at U2.N24 (DEC5): now also C11.2
- net at L1.1: now also C39.2, U4.D3 (LXB), U4.D4 (LXB)
- net 3.7V: now reaches BT1.1 (+)
- net 3.7V: now also C32.1, U4.A1 (BATT)
- net P0.02/AIN0 renamed AMUX
- net AMUX: now also U4.A4 (AMUX)
- net P0.06 renamed GPIO0
- net GPIO0: now also U4.A5 (GPIO0)
- net P0.07 renamed GPIO1
- net GPIO1: now also U4.A6 (GPIO1)
- net P0.08 renamed SCL
- net SCL: now also U4.D5 (SCL)
- net P0.18/RESET renamed nRST
- net nRST: now also R4.1, U4.B5 (NRST)
- net P0.26 renamed nIRQ
- net nIRQ: now also R3.1, U4.C5 (NIRQ)
- net P1.08 renamed SDA
- net SDA: now also U4.D6 (SDA)
- net VCC: no longer names the net of JP1.1
- net VCC: now also JP1.2
- new net: C31.1, U4.A2 (AVL), U4.B2 (PVL)
- new net: L1.2, U4.D1 (LXA), U4.D2 (LXA)
- new net: SW1.2, U4.B6 (NEN)
- new net: C13.1, L3.1, L4.2
- new net: C20.1, U4.E3 (SBB0)
- new net: C17.1, U4.C4 (SBB2)
- new net: C39.1, U4.E2 (BST)
- new net: C21.1, U4.E4 (SBB1)
- no-connect marks 15 -> 21
Other:
- note added: "1.0.0"
- note added: "IMU Breakout Holes"
- note added: "Power Management Circuit"
- note added: "TODO: How to use this?"
- note added: "TODO: Keep checking this stuff"
- note added: "Unused Outputs Do not leave unused outputs unconnected. If an output left unconnected is accidentally enabled, the charged inductor experiences an open circuit, and the output voltage soars above the absolute maximum rating, damaging the device. If an output is not used, do one of the following: 1. Disable the output (CNFG_SBBx_B.EN_SBBx[2:0] = 0x4 or 0x5) and connect the output to ground. If an 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"
- note removed: "${#}"
- note removed: "0.1.0"
- note removed: "D"
- note removed: "G"
- note removed: "I2C Pullups & Shift (IMU Breakout)"
- note removed: "IMU Breakout"
- note removed: "ON LED"
- note removed: "Optional"
- note removed: "Power Supply (Main)"
- note removed: "Power supply (IMU breakout)"
- note removed: "S"
- note removed: "STEMMA/I2C Headers (IMU Breakout)"
- moved on the sheet: BT1, JP1, JP2
