File: wearable/hw/prototype/prototype.kicad_sch (KiCad schematic)
At the start: 0 parts

Commit message: Prototype schematic done, organize repo a bit
Parts:
- added C1, C6, C7: 0.1uF, ECE445L:C_Axial_200mil, symbol ECE445L:C
- added C2: 1.5nF, ECE445L:C_Axial_200mil, symbol ECE445L:C
- added C3, C4, C8: 10uF, ECE445L:C_Axial_200mil, symbol ECE445L:C
- added C5: 1uF, ECE445L:C_Axial_200mil, symbol ECE445L:C
- added E1: ~, Connector_JST:JST_PH_S2B-PH-K_1x02_P2.00mm_Horizontal, symbol wearable:EEG_Electrode_Pair
- added EBIAS1: ~, Connector_PinHeader_1.00mm:PinHeader_1x01_P1.00mm_Vertical, symbol wearable:EEG_Electrode
- added R1, R10, R14, R2: 10k, symbol Device:R_US
- added R11, R15: 91k, symbol Device:R_US
- added R12: 330k, symbol Device:R_US
- added R13: 39k, symbol Device:R_US
- added R3, R4, R5, R6, R7, R9: 1M, symbol Device:R_US
- added R8: 4.7k, symbol Device:R_US
- added U1, U2: OPA2350, ECE445L:DIP-8_W7.62mm_LongPads, symbol ECE445L:OPA2350
- added U3: INA122P, PCM_Package_DIP_AKL:DIP-8_W7.62mm_LongPads, symbol PCM_Amplifier_Instrumentation_AKL:INA122P
Connections:
- new net: R3.2, R6.1, U3.2 (-)
- new net: C2.1, R5.1, R6.2, R7.2, U2.6 (-)
- new net: R1.2, R2.1, U1.3 (+)
- new net: R11.1, R13.1, U1.7
- new net: C6.1, R13.2, U2.2 (-)
- new net: EBIAS1.1, R9.1
- new net: C2.2, R5.2, R9.2, U2.7
- new net: E1.R, R4.1
- new net: R4.2, R7.1, U3.3 (+)
- new net: C5.2, R12.1, U1.6 (-)
- new net: R14.2, R15.2, U2.3 (+)
- new net: E1.L, R3.1
- new net: R8.1, U3.1 (RG)
- new net: R8.2, U3.8 (RG)
- new net: R10.2, R11.2, U1.5 (+)
- new net: C5.1, U3.6
- new net +3.3V: C1.1, C3.1, C4.1, C7.1, C8.1, R1.1, U1.8 (V+), U2.8 (V+), U3.7 (V+)
- new net GND: C4.2, C7.2, C8.2, R2.2, U1.4 (V-), U2.4 (V-), U3.4 (V-)
- new net P1.11: R15.1, U2.1
- new net VGND: C1.2, C3.2, C6.2, R10.1, R12.2, R14.1, U1.1, U1.2 (-), U2.5 (+), U3.5 (REF)
Other:
- note added: "Assembly Notes: -Isolate the analog inputs and output from eachother -IMPORTANT: make INA122P -> OPA2350_1.2 connection as short as possible -Twist the wires of the input pair to minimize EMI -Try to place bypass caps (the 0.1uF ones) as close as possible to the respective amp -See if a long ground rail free design is possible. i.e connect all ground pins close to the source. This will minimize n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"
- note added: "Design Notes: -This device uses only components from the checkout desk -We split up our filtering and amplifying into stages for better quality -INA122P: Grabs the voltage from the forehead while ignoring noise somewhat -OPA2350_1.1: Creates a virtual ground for the ADC to center around so the waves have room to go negative -OPA2350_1.2: Filters out DC components (HPF, fc = 0.5hz) -OPA2350_2.1: R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"
- note added: "WARNING: DO NOT RUN THIS SYSTEM PLUGGED INTO THE WALL. USE A BATTERY POWERED DEVICE (e.g. laptop) OR A BATTERY. YOU WILL GET FRIED OTHERWISE."

Commit message: Improved design guide
Other:
- note added: "FAQ: - I don't have a certain resistor/capacitor! What do I do! - All of these values *should* be at checkout desk, but if they aren't do some math to figure out a parallel or series combo that gets you within %5 tolerance."
Changed lines of the file:
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@@
+		)
+	)
+	(text "FAQ:\n- I don't have a certain resistor/capacitor! What do I do!\n	- All of these values *should* be at checkout desk, but if they aren't \n	do some math to figure out a parallel or series combo that gets you within %5 tolerance."
+		(exclude_from_sim no)
+		(at 75.438 133.096 0)
+		(effects
+			(font
+				(size 1.27 1.27)
+			)
+			(justify left)
 		)
 	)
